File: Frontend/kicad/FrontendPCBCoupon/FrontendPCBCoupon.kicad_sch (KiCad schematic)
At the start: 0 parts

Commit message: feat(kicad): coupon rev A - two-design staircase panel, per-piece grounds
The frontend PCB coupon, finished and ordered. 140.05 x 116.05 mm,
JLC04161H-7628 stackup (35 um / 0.2104 prepreg / In1 reference plane /
1.065 core / In2 / 0.2104 / 35 um, er 4.5).

Panel: seven coupon pieces self-panelised into two JLCPCB designs so
the order is billed as 2 unique boards instead of 7 (134 USD -> 84 USD).
Design 1 is a staircase, top to bottom: 90 mm line, directional coupler,
40 mm, 40 mm, 10 mm. Design 2 is the second coupler plus the vertical
90 mm line, their lower borders aligned. The two designs touch only
through 14 mouse bites (4 x 0.5 mm NPTH at 0.8 mm pitch) and a 2 mm
router slot; both pieces were verified separable - no stuck boundary
sample, every Edge.Cuts loop closed, no void touching the panel edge.

Connectors: all 18 SMAs are now BWSMA-KE-P001 edge mounts. The pads are
shorter than the Amphenol ones they replace, so every microstrip was
re-cut to keep the electrical length bit-identical: 90 / 40 / 40 / 10 /
90 mm through-lines and all eight coupler feeds at 23.4237 mm.

Grounds: one net per physical piece (GND_A .. GND_G, flattened to GND_1
and GND_2 on the two panelised designs) instead of a single GND, so the
pieces do not show up as unconnected islands. Plane zones merged to one
per piece per layer, 21 zones -> 6.

Thermal reliefs removed from every SMA ground pad (zone_connect 2).

DRC: 0 errors. 34 silk_over_copper warnings remain and are cosmetic -
16 of 18 refdes sit on bare copper, and all 14 information labels are
protected by F.Mask patches (checked by point-in-polygon).

Known risk, and the reason this coupon exists: the coupler comb fingers
are 0.100 mm wide with 0.100 mm gaps, against a JLC minimum of 0.09 mm,
so a +/-20 % etch tolerance lands on the edge of the process.

panel/ holds the generator: gen.py builds the rectilinear union of the
piece outlines by coordinate compression and boundary tracing, emit.py
writes Edge.Cuts with R = 1.0 mm r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
Parts:
- added J1, J10, J11, J12, J13, J14, J15, J16, J17, J18, J2, J3, J4, J5, J6, J7, J8, J9: BWSMA-KE-P001, Frontend:SMA_BWSMA-KE-P001_EdgeMount, symbol Frontend:SMA_BWSMA-KE-P001
- added PD1, PD2: Dir Coupler (C=15dB), Frontend:FunRad_Coupler_5GHz8_Symmetric_15dB, symbol Frontend:DirCoupler
Connections:
- new net: J17.1 (In), J18.1 (In)
- new net: J7.1 (In), PD1.1 (In)
- new net: J15.1 (In), J16.1 (In)
- new net: J1.1 (In), J2.1 (In)
- new net: J5.1 (In), J6.1 (In)
- new net: J14.1 (In), PD2.4 (Isolated)
- new net: J3.1 (In), J4.1 (In)
- new net: J11.1 (In), PD2.1 (In)
- new net: J13.1 (In), PD2.2 (Thru)
- new net: J12.1 (In), PD2.3 (Coupled)
- new net: J9.1 (In), PD1.2 (Thru)
- new net: J10.1 (In), PD1.4 (Isolated)
- new net: J8.1 (In), PD1.3 (Coupled)
- new net GND_1: J1.2 (Ext), J10.2 (Ext), J15.2 (Ext), J16.2 (Ext), J2.2 (Ext), J3.2 (Ext), J4.2 (Ext), J5.2 (Ext), J6.2 (Ext), J7.2 (Ext), J8.2 (Ext), J9.2 (Ext)
- new net GND_2: J11.2 (Ext), J12.2 (Ext), J13.2 (Ext), J14.2 (Ext), J17.2 (Ext), J18.2 (Ext)
